Commit message: Updated Xacro file

File: src/servo/servo_description/urdf/servo.xacro (robot description, xacro)
@@ -10,4 +10,9 @@
   <xacro:property name="width" value="0.1" /> <!-- width of the beam -->
   <xacro:property name="offset" value="0" /> <!-- width of the beam -->
+  <xacro:property name="spacing" value="0.25" /> <!-- width of the beam -->
+  <xacro:property name="leftmost" value="-0.2" /> <!-- leftmost y cordinate of palm -->
+  <xacro:property name="imr_width" value="0.173" /> <!-- index middle ring width -->
+  <xacro:property name="l_width" value="0.15" /> <!-- little width -->
+  <xacro:property name="x_width" value="0.10" /> <!-- little width -->
   <xacro:include filename="$(find servo_description)/urdf/servo.gazebo" />
   <xacro:include filename="$(find servo_description)/urdf/materials.xacro" />
@@ -15,18 +20,18 @@
   <link name="Palm">
     <collision>
-      <origin xyz="0 0.15 0.5" rpy="0 0 0"/>
-      <geometry>
-         <box size="0.15 0.7 1"/>
-      </geometry>
-    </collision>
-    <visual>
-      <origin xyz="0 0.15 0.5" rpy="0 0 0"/>
-      <geometry>
-         <box size="0.15 0.7 1"/>
+      <origin xyz="0 ${(leftmost+imr_width/2+spacing*3+l_width/2+leftmost)/2} 0.5" rpy="0 0 0"/>
+      <geometry>
+         <box size="${x_width*2} ${(leftmost+imr_width/2+spacing*3+l_width/2+leftmost)+0.4} 1"/>
+      </geometry>
+    </collision>
+    <visual>
+      <origin xyz="0 ${(leftmost+imr_width/2+spacing*3+l_width/2+leftmost)/2} 0.5" rpy="0 0 0"/>
+      <geometry>
+         <box size="${x_width*2} ${(leftmost+imr_width/2+spacing*3+l_width/2+leftmost)+0.4} 1"/>
       </geometry>
       <material name="skin"/>
     </visual>
     <inertial>
-      <origin xyz="0 0.15 0.5" rpy="0 0 0"/>
+      <origin xyz="0 ${(leftmost+imr_width/2+spacing*3+l_width/2+leftmost)/2} 0.5" rpy="0 0 0"/>
       <mass value="${mass1}"/>
       <inertia
@@ -40,43 +45,43 @@
     <parent link="Palm"/>
     <child link="segt1"/>
-    <origin xyz="0 -0.25 0.1" rpy="0.52 0 0"/>
+    <origin xyz="0 ${leftmost-0.05} 0.3" rpy="0.52 0 0"/>
   </joint>
   <joint name="jointG1" type="fixed">
     <parent link="Palm"/>
     <child link="seg11"/>
-    <origin xyz="0 -0.15 1" rpy="0 0 0"/>
+    <origin xyz="0 ${leftmost+imr_width/2} 1" rpy="0 0 0"/>
   </joint>
   <joint name="jointG2" type="fixed">
     <parent link="Palm"/>
     <child link="seg21"/>
-    <origin xyz="0 0.05 1" rpy="0 0 0"/>
+    <origin xyz="0 ${leftmost+imr_width/2+spacing} 1" rpy="0 0 0"/>
   </joint>
   <joint name="jointG3" type="fixed">
     <parent link="Palm"/>
     <child link="seg31"/>
-    <origin xyz="0 0.25 1" rpy="0 0 0"/>
+    <origin xyz="0 ${leftmost+imr_width/2+spacing*2} 1" rpy="0 0 0"/>
   </joint>
   <joint name="jointG4" type="fixed">
     <parent link="Palm"/>
     <child link="seg41"/>
-    <origin xyz="0 0.45 1" rpy="0 0 0"/>
+    <origin xyz="0 ${leftmost+imr_width/2+spacing*3} 1" rpy="0 0 0"/>
   </joint>
 <!--====================== THUMB ===============================-->
   <link name="segt1">
     <collision>
-      <origin xyz="0 0 0.25" rpy="0 0 0"/>
-      <geometry>
-         <box size="0.1 0.1 0.5"/>
-      </geometry>
-    </collision>
-    <visual>
-      <origin xyz="0 0 0.25" rpy="0 0 0"/>
-      <geometry>
-         <box size="0.1 0.1 0.5"/>
+      <origin xyz="0 0 ${0.15/2}" rpy="0 0 0"/>
+      <geometry>
+         <box size="${x_width} 0.21 0.15"/>
+      </geometry>
+    </collision>
+    <visual>
+      <origin xyz="0 0 ${0.15/2}" rpy="0 0 0"/>
+      <geometry>
+         <box size="${x_width} 0.21 0.15"/>
       </geometry>
       <material name="orange"/>
     </visual>
     <inertial>
-      <origin xyz="0 0 0.25" rpy="0 0 0"/>
+      <origin xyz="0 0 ${0.15/2}" rpy="0 0 0"/>
       <mass value="${mass1}"/>
       <inertia
@@ -89,5 +94,5 @@
     <parent link="segt1"/>
     <child link="segt2"/>
-    <origin xyz="0.05 0 0.5" rpy="0 0 0"/>
+    <origin xyz="${x_width/2} 0 0.15" rpy="0 0 0"/>
     <axis xyz="0 1 0"/>
     <dynamics damping="0.7"/>
@@ -96,18 +101,18 @@
   <link name="segt2">
     <collision>
-      <origin xyz="-0.05 0 0.25" rpy="0 0 0"/>
-      <geometry>
-         <box size="0.1 0.1 0.5"/>
-      </geometry>
-    </collision>
-    <visual>
-      <origin xyz="-0.05 0 0.25" rpy="0 0 0"/>
-      <geometry>
-         <box size="0.1 0.1 0.5"/>
-      </geometry>
-      <material name="black"/>
-    </visual>
-    <inertial>
-      <origin xyz="-0.05 0 0.25" rpy="0 0 0"/>
+      <origin xyz="${-x_width/2} 0 ${0.268/2}" rpy="0 0 0"/>
+      <geometry>
+         <box size="${x_width} 0.21 0.268"/>
+      </geometry>
+    </collision>
+    <visual>
+      <origin xyz="${-x_width/2} 0 ${0.268/2}" rpy="0 0 0"/>
+      <geometry>
+         <box size="${x_width} 0.21 0.268"/>
+      </geometry>
+      <material name="black"/>
+    </visual>
+    <inertial>
+      <origin xyz="${-x_width/2} 0 ${0.268/2}" rpy="0 0 0"/>
       <mass value="${mass}"/>
       <inertia
@@ -120,5 +125,5 @@
     <parent link="segt2"/>
     <child link="segt3"/>
-    <origin xyz="0 0 0.5" rpy="0 0 0"/>
+    <origin xyz="0 0 ${0.268}" rpy="0 0 0"/>
     <axis xyz="0 1 0"/>
     <dynamics damping="0.7"/>
@@ -127,18 +132,18 @@
   <link name="segt3">
     <collision>
-      <origin xyz="-0.05 0 0.25" rpy="0 0 0"/>
-      <geometry>
-         <box size="0.1 0.1 0.5"/>
-      </geometry>
-    </collision>
-    <visual>
-      <origin xyz="-0.05 0 0.25" rpy="0 0 0"/>
-      <geometry>
-         <box size="0.1 0.1 0.5"/>
-      </geometry>
-      <material name="black"/>
-    </visual>
-    <inertial>
-      <origin xyz="-0.05 0 0.25" rpy="0 0 0"/>
+      <origin xyz="${-x_width/2} 0 ${0.268/2}" rpy="0 0 0"/>
+      <geometry>
+         <box size="${x_width} 0.21 0.268"/>
+      </geometry>
+    </collision>
+    <visual>
+      <origin xyz="${-x_width/2} 0 ${0.268/2}" rpy="0 0 0"/>
+      <geometry>
+         <box size="${x_width} 0.21 0.268"/>
+      </geometry>
+      <material name="black"/>
+    </visual>
+    <inertial>
+      <origin xyz="${-x_width/2} 0 ${0.268/2}" rpy="0 0 0"/>
       <mass value="${mass}"/>
       <inertia
@@ -151,18 +156,18 @@
   <link name="seg11">
     <collision>
-      <origin xyz="0 0 0.25" rpy="0 0 0"/>
-      <geometry>
-	       <box size="0.1 0.1 0.5"/>
-      </geometry>
-    </collision>
-    <visual>
-      <origin xyz="0 0 0.25" rpy="0 0 0"/>
-      <geometry>
-	       <box size="0.1 0.1 0.5"/>
+      <origin xyz="0 0 ${0.268/2}" rpy="0 0 0"/>
+      <geometry>
+	       <box size="${x_width} ${imr_width} 0.268"/>
+      </geometry>
+    </collision>
+    <visual>
+      <origin xyz="0 0 ${0.268/2}" rpy="0 0 0"/>
+      <geometry>
+	       <box size="${x_width} ${imr_width} 0.268"/>
       </geometry>
       <material name="orange"/>
     </visual>
     <inertial>
-      <origin xyz="0 0 0.25" rpy="0 0 0"/>
+      <origin xyz="0 0 ${0.268/2}" rpy="0 0 0"/>
       <mass value="${mass1}"/>
       <inertia
@@ -175,5 +180,5 @@
     <parent link="seg11"/>
     <child link="seg12"/>
-    <origin xyz="0.05 0 0.5" rpy="0 0 0"/>
+    <origin xyz="${x_width/2} 0 0.268" rpy="0 0 0"/>
     <axis xyz="0 1 0"/>
     <dynamics damping="0.7"/>
@@ -182,18 +187,18 @@
   <link name="seg12">
     <collision>
-      <origin xyz="-0.05 0 0.25" rpy="0 0 0"/>
-      <geometry>
-	       <box size="0.1 0.1 0.5"/>
-      </geometry>
-    </collision>
-    <visual>
-      <origin xyz="-0.05 0 0.25" rpy="0 0 0"/>
-      <geometry>
-	       <box size="0.1 0.1 0.5"/>
-      </geometry>
-      <material name="black"/>
-    </visual>
-    <inertial>
-      <origin xyz="-0.05 0 0.25" rpy="0 0 0"/>
+      <origin xyz="${-x_width/2} 0 ${0.268/2}" rpy="0 0 0"/>
+      <geometry>
+	       <box size="${x_width} ${imr_width} 0.268"/>
+      </geometry>
+    </collision>
+    <visual>
+      <origin xyz="${-x_width/2} 0 ${0.268/2}" rpy="0 0 0"/>
+      <geometry>
+	       <box size="${x_width} ${imr_width} 0.268"/>
+      </geometry>
+      <material name="black"/>
+    </visual>
+    <inertial>
+      <origin xyz="${-x_width/2} 0 ${0.268/2}" rpy="0 0 0"/>
       <mass value="${mass}"/>
       <inertia
@@ -206,5 +211,5 @@
     <parent link="seg12"/>
     <child link="seg13"/>
-    <origin xyz="0 0 0.5" rpy="0 0 0"/>
+    <origin xyz="0 0 ${0.268}" rpy="0 0 0"/>
     <axis xyz="0 1 0"/>
     <dynamics damping="0.7"/>
@@ -213,18 +218,18 @@
   <link name="seg13">
     <collision>
-      <origin xyz="-0.05 0 0.25" rpy="0 0 0"/>
-      <geometry>
-         <box size="0.1 0.1 0.5"/>
-      </geometry>
-    </collision>
-    <visual>
-      <origin xyz="-0.05 0 0.25" rpy="0 0 0"/>
-      <geometry>
-         <box size="0.1 0.1 0.5"/>
-      </geometry>
-      <material name="black"/>
-    </visual>
-    <inertial>
-      <origin xyz="-0.05 0 0.25" rpy="0 0 0"/>
+      <origin xyz="${-x_width/2} 0 ${0.268/2}" rpy="0 0 0"/>
+      <geometry>
+         <box size="${x_width} ${imr_width} 0.268"/>
+      </geometry>
+    </collision>
+    <visual>
+      <origin xyz="${-x_width/2} 0 ${0.268/2}" rpy="0 0 0"/>
+      <geometry>
+         <box size="${x_width} ${imr_width} 0.268"/>
+      </geometry>
+      <material name="black"/>
+    </visual>
+    <inertial>
+      <origin xyz="${-x_width/2} 0 ${0.268/2}" rpy="0 0 0"/>
       <mass value="${mass}"/>
       <inertia
@@ -237,18 +242,18 @@
   <link name="seg21">
     <collision>
-      <origin xyz="0.0 0.0 0.25" rpy="0 0 0"/>
-      <geometry>
-         <box size="0.1 0.1 0.5"/>
-      </geometry>
-    </collision>
-    <visual>
-      <origin xyz="0.0 0.0 0.25" rpy="0 0 0"/>
-      <geometry>
-         <box size="0.1 0.1 0.5"/>
+      <origin xyz="0 0 ${0.3/2}" rpy="0 0 0"/>
+      <geometry>
+         <box size="${x_width} ${imr_width} 0.2"/>
+      </geometry>
+    </collision>
+    <visual>
+      <origin xyz="0 0 ${0.3/2}" rpy="0 0 0"/>
+      <geometry>
+         <box size="${x_width} ${imr_width} 0.3"/>
       </geometry>
       <material name="orange"/>
     </visual>
     <inertial>
-      <origin xyz="0.0 0.0 0.25" rpy="0 0 0"/>
+      <origin xyz="0 0 ${0.3/2}" rpy="0 0 0"/>
       <mass value="${mass1}"/>
       <inertia
@@ -261,5 +266,5 @@
     <parent link="seg21"/>
     <child link="seg22"/>
-    <origin xyz="0.05 0.0 0.5" rpy="0 0 0"/>
+    <origin xyz="${x_width/2} 0.0 0.3" rpy="0 0 0"/>
     <axis xyz="0 1 0"/>
     <dynamics damping="0.7"/>
@@ -268,18 +273,18 @@
   <link name="seg22">
     <collision>
-      <origin xyz="-0.05 0 0.25" rpy="0 0 0"/>
-      <geometry>
-         <box size="0.1 0.1 0.5"/>
-      </geometry>
-    </collision>
-    <visual>
-      <origin xyz="-0.05 0 0.25" rpy="0 0 0"/>
-      <geometry>
-         <box size="0.1 0.1 0.5"/>
-      </geometry>
-      <material name="black"/>
-    </visual>
-    <inertial>
-      <origin xyz="-0.05 0 0.25" rpy="0 0 0"/>
+      <origin xyz="${-x_width/2} 0 ${0.3/2}" rpy="0 0 0"/>
+      <geometry>
+         <box size="${x_width} ${imr_width} 0.3"/>
+      </geometry>
+    </collision>
+    <visual>
+      <origin xyz="${-x_width/2} 0 ${0.3/2}" rpy="0 0 0"/>
+      <geometry>
+         <box size="${x_width} ${imr_width} 0.3"/>
+      </geometry>
+      <material name="black"/>
+    </visual>
+    <inertial>
+      <origin xyz="${-x_width/2} 0 ${0.3/2}" rpy="0 0 0"/>
       <mass value="${mass}"/>
       <inertia
@@ -292,5 +297,5 @@
     <parent link="seg22"/>
     <child link="seg23"/>
-    <origin xyz="0 0 0.5" rpy="0 0 0"/>
+    <origin xyz="0 0 0.3" rpy="0 0 0"/>
     <axis xyz="0 1 0"/>
     <dynamics damping="0.7"/>
@@ -299,18 +304,18 @@
   <link name="seg23">
     <collision>
-      <origin xyz="-0.05 0 0.25" rpy="0 0 0"/>
-      <geometry>
-         <box size="0.1 0.1 0.5"/>
-      </geometry>
-    </collision>
-    <visual>
-      <origin xyz="-0.05 0 0.25" rpy="0 0 0"/>
-      <geometry>
-         <box size="0.1 0.1 0.5"/>
-      </geometry>
-      <material name="black"/>
-    </visual>
-    <inertial>
-      <origin xyz="-0.05 0 0.25" rpy="0 0 0"/>
+      <origin xyz="${-x_width/2} 0 ${0.3/2}" rpy="0 0 0"/>
+      <geometry>
+         <box size="${x_width} ${imr_width} 0.3"/>
+      </geometry>
+    </collision>
+    <visual>
+      <origin xyz="${-x_width/2} 0 ${0.3/2}" rpy="0 0 0"/>
+      <geometry>
+         <box size="${x_width} ${imr_width} 0.3"/>
+      </geometry>
+      <material name="black"/>
+    </visual>
+    <inertial>
+      <origin xyz="${-x_width/2} 0 ${0.3/2}" rpy="0 0 0"/>
       <mass value="${mass}"/>
       <inertia
@@ -323,18 +328,18 @@
   <link name="seg31">
     <collision>
-      <origin xyz="0.0 0 0.25" rpy="0 0 0"/>
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