Commit message: Added hand joints and unfixed controllers

File: src/servo/servo_description/urdf/servo.xacro (robot description, xacro)
@@ -3,6 +3,6 @@
   <!-- Constants for robot dimensions -->
   <xacro:property name="PI" value="3.1415926535897931"/>
-  <xacro:property name="mass" value="1" /> <!-- arbitrary value for mass -->
-  <xacro:property name="mass1" value="5000" /> <!-- arbitrary value for mass -->
+  <xacro:property name="mass_palm" value="0.2" /> <!-- arbitrary value for mass -->
+  <xacro:property name="mass_hand" value="20" /> <!-- arbitrary value for mass -->
   <xacro:property name="radius" value="0.05" /> <!-- Radii of the cylinder-->
   <xacro:property name="length1" value="0.1" /> <!-- seg42 -->
@@ -14,7 +14,107 @@
   <xacro:property name="imr_width" value="0.173" /> <!-- index middle ring width -->
   <xacro:property name="l_width" value="0.15" /> <!-- little width -->
-  <xacro:property name="x_width" value="0.10" /> <!-- little width -->
+  <xacro:property name="x_width" value="0.10" />
+  <xacro:property name="hand_height" value="3" /> <!-- little width -->
+  <xacro:property name="hand_radius" value="0.30" /> <!-- little width -->
   <xacro:include filename="$(find servo_description)/urdf/servo.gazebo" />
   <xacro:include filename="$(find servo_description)/urdf/materials.xacro" />
+<!--======================= Right Hand =================================== -->
+  <link name="Right_upper">
+    <collision>
+      <origin xyz="0 0 ${hand_height/2}" rpy="0 0 0"/>
+      <geometry>
+         <cylinder length="${hand_height}" radius="${hand_radius}"/>
+      </geometry>
+    </collision>
+    <visual>
+      <origin xyz="0 0 ${hand_height/2}" rpy="0 0 0"/>
+      <geometry>
+         <cylinder length="${hand_height}" radius="${hand_radius}"/>
+      </geometry>
+    </visual>
+    <inertial>
+      <origin xyz="0 0 ${hand_height/2}" rpy="0 0 0"/>
+      <mass value="${mass_hand*1000}"/>
+      <inertia
+          ixx="${1/12*mass_hand*hand_height*hand_height}" ixy="0.0" ixz="0.0"
+          iyy="${1/12*mass_hand*hand_height*hand_height}" iyz="0.0"
+          izz="${mass_hand*radius*radius}"/>
+    </inertial>
+  </link>
+  <joint name="Right_hinge" type="revolute">
+    <parent link="Right_upper"/>
+    <child link="Right_lower"/>
+    <origin xyz="${hand_radius} 0 ${hand_height}" rpy="0 0 0"/>
+    <axis xyz="0 1 0"/>
+    <dynamics damping="0.9"/>
+    <limit effort="1000.0" lower="0" upper="1.57" velocity="10"/>
+  </joint>
+  <link name="Right_lower">
+     <collision>
+      <origin xyz="${-hand_radius} 0 ${hand_height/2}" rpy="0 0 0"/>
+      <geometry>
+         <cylinder length="${hand_height}" radius="${hand_radius}"/>
+      </geometry>
+    </collision>
+    <visual>
+      <origin xyz="${-hand_radius} 0 ${hand_height/2}" rpy="0 0 0"/>
+      <geometry>
+         <cylinder length="${hand_height}" radius="${hand_radius}"/>
+      </geometry>
+    </visual>
+    <inertial>
+      <origin xyz="${-hand_radius} 0 ${hand_height/2}" rpy="0 0 0"/>
+      <mass value="${mass_hand}"/>
+      <inertia
+          ixx="${1/12*mass_hand*hand_height*hand_height}" ixy="0.0" ixz="0.0"
+          iyy="${1/12*mass_hand*hand_height*hand_height}" iyz="0.0"
+          izz="${mass_hand*radius*radius}"/>
+    </inertial>
+  </link>
+<!-- ===============3 axis PALM joint ======================================= -->
+  <joint name="Right_palm_y" type="revolute">
+    <parent link="Right_lower"/>
+    <child link="Right_z_palmD"/>
+    <origin xyz="${-hand_radius} ${-(leftmost+imr_width/2+spacing*3+l_width/2+leftmost)/2} ${hand_height}" rpy="0 0 0"/>
+    <axis xyz="0 1 0"/>
+    <dynamics damping="0.7"/>
+    <limit effort="1000.0" lower="-1.57" upper="1.57" velocity="10"/>
+  </joint>
+  <link name="Right_z_palmD"> <!-- https://answers.ros.org/question/258420/ball-joint-in-urdf/ -->
+    <inertial>
+      <mass value="0.00025" />
+      <inertia ixx="5.8083e-4" ixy="0" ixz="0" iyy="3.0833e-5" iyz="0" izz="5.9083e-4" />
+    </inertial>
+  </link>
+  <joint name="Right_palm_z" type="revolute">
+    <parent link="Right_z_palmD"/>
+    <child link="Right_x_palmD"/>
+    <axis xyz="0 0 1"/>
+    <dynamics damping="0.7"/>
+    <limit effort="1000.0" lower="-1.57" upper="1.57" velocity="10"/>
+  </joint>
+  <link name="Right_x_palmD">
+    <inertial>
+      <mass value="0.00025" />
+      <inertia ixx="5.8083e-4" ixy="0" ixz="0" iyy="3.0833e-5" iyz="0" izz="5.9083e-4" />
+    </inertial>
+  </link>
+  <joint name="Right_palm_x" type="revolute">
+    <parent link="Right_x_palmD"/>
+    <child link="Right_y_palmD"/>
+    <axis xyz="1 0 0"/>
+    <dynamics damping="0.7"/>
+    <limit effort="1000.0" lower="-1.57" upper="1.57" velocity="10"/>
+  </joint>
+  <link name="Right_y_palmD">
+    <inertial>
+      <mass value="0.00025" />
+      <inertia ixx="5.8083e-4" ixy="0" ixz="0" iyy="3.0833e-5" iyz="0" izz="5.9083e-4" />
+    </inertial>
+  </link>
+  <joint name="Right_palm_d" type="fixed">
+    <parent link="Right_y_palmD"/>
+    <child link="Palm"/>
+  </joint>
 <!--========================PALM ========================================= -->
   <link name="Palm">
@@ -34,10 +134,10 @@
     <inertial>
       <origin xyz="0 ${(leftmost+imr_width/2+spacing*3+l_width/2+leftmost)/2} 0.5" rpy="0 0 0"/>
-      <mass value="${mass1}"/>
-      <inertia
-          ixx="${mass1 / 12.0 * (length1*length1 + length1*length1)}" ixy="0.0" ixz="0.0"
-          iyy="${mass1 / 12.0 * (length1*length1 + length1*length1)}" iyz="0.0"
-          izz="${mass1 / 12.0 * (length1*length1 + length1*length1)}"/>
-      </inertial>
+      <mass value="${mass_palm}"/>
+      <inertia
+          ixx="${mass_palm / 12.0 * (length1*length1 + length1*length1)}" ixy="0.0" ixz="0.0"
+          iyy="${mass_palm / 12.0 * (length1*length1 + length1*length1)}" iyz="0.0"
+          izz="${mass_palm / 12.0 * (length1*length1 + length1*length1)}"/>
+    </inertial>
   </link>
 <!--========================PALM JOINTS ========================================= -->
@@ -84,9 +184,9 @@
     <inertial>
       <origin xyz="0 0 ${0.15/2}" rpy="0 0 0"/>
-      <mass value="${mass1}"/>
-      <inertia
-    ixx="${mass1 / 12.0 * (length1*length1 + length1*length1)}" ixy="0.0" ixz="0.0"
-    iyy="${mass1 / 12.0 * (length1*length1 + length1*length1)}" iyz="0.0"
-    izz="${mass1 / 12.0 * (length1*length1 + length1*length1)}"/>
+      <mass value="${mass_palm}"/>
+      <inertia
+    ixx="${mass_palm / 12.0 * (length1*length1 + length1*length1)}" ixy="0.0" ixz="0.0"
+    iyy="${mass_palm / 12.0 * (length1*length1 + length1*length1)}" iyz="0.0"
+    izz="${mass_palm / 12.0 * (length1*length1 + length1*length1)}"/>
     </inertial>
   </link>
@@ -115,9 +215,9 @@
     <inertial>
       <origin xyz="${-x_width/2} 0 ${0.268/2}" rpy="0 0 0"/>
-      <mass value="${mass}"/>
-      <inertia
-    ixx="${mass / 12.0 * (width*width + width*width)}" ixy="0.0" ixz="0.0"
-    iyy="${mass / 12.0 * (length2*length2 + width*width)}" iyz="0.0"
-    izz="${mass / 12.0 * (width*width + length2*length2)}"/>
+      <mass value="${mass_palm}"/>
+      <inertia
+    ixx="${mass_palm / 12.0 * (width*width + width*width)}" ixy="0.0" ixz="0.0"
+    iyy="${mass_palm / 12.0 * (length2*length2 + width*width)}" iyz="0.0"
+    izz="${mass_palm / 12.0 * (width*width + length2*length2)}"/>
     </inertial>
   </link>
@@ -146,9 +246,9 @@
     <inertial>
       <origin xyz="${-x_width/2} 0 ${0.268/2}" rpy="0 0 0"/>
-      <mass value="${mass}"/>
-      <inertia
-    ixx="${mass / 12.0 * (width*width + width*width)}" ixy="0.0" ixz="0.0"
-    iyy="${mass / 12.0 * (length2*length2 + width*width)}" iyz="0.0"
-    izz="${mass / 12.0 * (width*width + length2*length2)}"/>
+      <mass value="${mass_palm}"/>
+      <inertia
+    ixx="${mass_palm / 12.0 * (width*width + width*width)}" ixy="0.0" ixz="0.0"
+    iyy="${mass_palm / 12.0 * (length2*length2 + width*width)}" iyz="0.0"
+    izz="${mass_palm / 12.0 * (width*width + length2*length2)}"/>
     </inertial>
   </link>
@@ -170,9 +270,9 @@
     <inertial>
       <origin xyz="0 0 ${0.268/2}" rpy="0 0 0"/>
-      <mass value="${mass1}"/>
-      <inertia
-	  ixx="${mass1 / 12.0 * (length1*length1 + length1*length1)}" ixy="0.0" ixz="0.0"
-	  iyy="${mass1 / 12.0 * (length1*length1 + length1*length1)}" iyz="0.0"
-	  izz="${mass1 / 12.0 * (length1*length1 + length1*length1)}"/>
+      <mass value="${mass_palm}"/>
+      <inertia
+	  ixx="${mass_palm / 12.0 * (length1*length1 + length1*length1)}" ixy="0.0" ixz="0.0"
+	  iyy="${mass_palm / 12.0 * (length1*length1 + length1*length1)}" iyz="0.0"
+	  izz="${mass_palm / 12.0 * (length1*length1 + length1*length1)}"/>
     </inertial>
   </link>
@@ -201,9 +301,9 @@
     <inertial>
       <origin xyz="${-x_width/2} 0 ${0.268/2}" rpy="0 0 0"/>
-      <mass value="${mass}"/>
-      <inertia
-	  ixx="${mass / 12.0 * (width*width + width*width)}" ixy="0.0" ixz="0.0"
-	  iyy="${mass / 12.0 * (length2*length2 + width*width)}" iyz="0.0"
-	  izz="${mass / 12.0 * (width*width + length2*length2)}"/>
+      <mass value="${mass_palm}"/>
+      <inertia
+	  ixx="${mass_palm / 12.0 * (width*width + width*width)}" ixy="0.0" ixz="0.0"
+	  iyy="${mass_palm / 12.0 * (length2*length2 + width*width)}" iyz="0.0"
+	  izz="${mass_palm / 12.0 * (width*width + length2*length2)}"/>
     </inertial>
   </link>
@@ -232,9 +332,9 @@
     <inertial>
       <origin xyz="${-x_width/2} 0 ${0.268/2}" rpy="0 0 0"/>
-      <mass value="${mass}"/>
-      <inertia
-    ixx="${mass / 12.0 * (width*width + width*width)}" ixy="0.0" ixz="0.0"
-    iyy="${mass / 12.0 * (length2*length2 + width*width)}" iyz="0.0"
-    izz="${mass / 12.0 * (width*width + length2*length2)}"/>
+      <mass value="${mass_palm}"/>
+      <inertia
+    ixx="${mass_palm / 12.0 * (width*width + width*width)}" ixy="0.0" ixz="0.0"
+    iyy="${mass_palm / 12.0 * (length2*length2 + width*width)}" iyz="0.0"
+    izz="${mass_palm / 12.0 * (width*width + length2*length2)}"/>
     </inertial>
   </link>
@@ -256,9 +356,9 @@
     <inertial>
       <origin xyz="0 0 ${0.3/2}" rpy="0 0 0"/>
-      <mass value="${mass1}"/>
-      <inertia
-    ixx="${mass1 / 12.0 * (length1*length1 + length1*length1)}" ixy="0.0" ixz="0.0"
-    iyy="${mass1 / 12.0 * (length1*length1 + length1*length1)}" iyz="0.0"
-    izz="${mass1 / 12.0 * (length1*length1 + length1*length1)}"/>
+      <mass value="${mass_palm}"/>
+      <inertia
+    ixx="${mass_palm / 12.0 * (length1*length1 + length1*length1)}" ixy="0.0" ixz="0.0"
+    iyy="${mass_palm / 12.0 * (length1*length1 + length1*length1)}" iyz="0.0"
+    izz="${mass_palm / 12.0 * (length1*length1 + length1*length1)}"/>
     </inertial>
   </link>
@@ -287,9 +387,9 @@
     <inertial>
       <origin xyz="${-x_width/2} 0 ${0.3/2}" rpy="0 0 0"/>
-      <mass value="${mass}"/>
-      <inertia
-    ixx="${mass / 12.0 * (width*width + width*width)}" ixy="0.0" ixz="0.0"
-    iyy="${mass / 12.0 * (length2*length2 + width*width)}" iyz="0.0"
-    izz="${mass / 12.0 * (width*width + length2*length2)}"/>
+      <mass value="${mass_palm}"/>
+      <inertia
+    ixx="${mass_palm / 12.0 * (width*width + width*width)}" ixy="0.0" ixz="0.0"
+    iyy="${mass_palm / 12.0 * (length2*length2 + width*width)}" iyz="0.0"
+    izz="${mass_palm / 12.0 * (width*width + length2*length2)}"/>
     </inertial>
   </link>
@@ -318,9 +418,9 @@
     <inertial>
       <origin xyz="${-x_width/2} 0 ${0.3/2}" rpy="0 0 0"/>
-      <mass value="${mass}"/>
-      <inertia
-    ixx="${mass / 12.0 * (width*width + width*width)}" ixy="0.0" ixz="0.0"
-    iyy="${mass / 12.0 * (length2*length2 + width*width)}" iyz="0.0"
-    izz="${mass / 12.0 * (width*width + length2*length2)}"/>
+      <mass value="${mass_palm}"/>
+      <inertia
+    ixx="${mass_palm / 12.0 * (width*width + width*width)}" ixy="0.0" ixz="0.0"
+    iyy="${mass_palm / 12.0 * (length2*length2 + width*width)}" iyz="0.0"
+    izz="${mass_palm / 12.0 * (width*width + length2*length2)}"/>
     </inertial>
   </link>
@@ -342,9 +442,9 @@
     <inertial>
       <origin xyz="0 0 ${0.24/2}" rpy="0 0 0"/>
-      <mass value="${mass1}"/>
-      <inertia
-    ixx="${mass1 / 12.0 * (length1*length1 + length1*length1)}" ixy="0.0" ixz="0.0"
-    iyy="${mass1 / 12.0 * (length1*length1 + length1*length1)}" iyz="0.0"
-    izz="${mass1 / 12.0 * (length1*length1 + length1*length1)}"/>
+      <mass value="${mass_palm}"/>
+      <inertia
+    ixx="${mass_palm / 12.0 * (length1*length1 + length1*length1)}" ixy="0.0" ixz="0.0"
+    iyy="${mass_palm / 12.0 * (length1*length1 + length1*length1)}" iyz="0.0"
+    izz="${mass_palm / 12.0 * (length1*length1 + length1*length1)}"/>
     </inertial>
   </link>
@@ -373,9 +473,9 @@
     <inertial>
       <origin xyz="${-x_width/2} 0 ${0.24/2}" rpy="0 0 0"/>
-      <mass value="${mass}"/>
-      <inertia
-    ixx="${mass / 12.0 * (width*width + width*width)}" ixy="0.0" ixz="0.0"
-    iyy="${mass / 12.0 * (length2*length2 + width*width)}" iyz="0.0"
-    izz="${mass / 12.0 * (width*width + length2*length2)}"/>
+      <mass value="${mass_palm}"/>
+      <inertia
+    ixx="${mass_palm / 12.0 * (width*width + width*width)}" ixy="0.0" ixz="0.0"
+    iyy="${mass_palm / 12.0 * (length2*length2 + width*width)}" iyz="0.0"
+    izz="${mass_palm / 12.0 * (width*width + length2*length2)}"/>
     </inertial>
   </link>
@@ -404,9 +504,9 @@
     <inertial>
       <origin xyz="${-x_width/2} 0 ${0.24/2}" rpy="0 0 0"/>
-      <mass value="${mass}"/>
-      <inertia
-    ixx="${mass / 12.0 * (width*width + width*width)}" ixy="0.0" ixz="0.0"
-    iyy="${mass / 12.0 * (length2*length2 + width*width)}" iyz="0.0"
-    izz="${mass / 12.0 * (width*width + length2*length2)}"/>
+      <mass value="${mass_palm}"/>
+      <inertia
+    ixx="${mass_palm / 12.0 * (width*width + width*width)}" ixy="0.0" ixz="0.0"
+    iyy="${mass_palm / 12.0 * (length2*length2 + width*width)}" iyz="0.0"
+    izz="${mass_palm / 12.0 * (width*width + length2*length2)}"/>
     </inertial>
   </link>
@@ -428,9 +528,9 @@
     <inertial>
       <origin xyz="0 0 ${0.15/2}" rpy="0 0 0"/>
-      <mass value="${mass1}"/>
-      <inertia
-    ixx="${mass1 / 12.0 * (length1*length1 + length1*length1)}" ixy="0.0" ixz="0.0"
-    iyy="${mass1 / 12.0 * (length1*length1 + length1*length1)}" iyz="0.0"
-    izz="${mass1 / 12.0 * (length1*length1 + length1*length1)}"/>
+      <mass value="${mass_palm}"/>
+      <inertia
+    ixx="${mass_palm / 12.0 * (length1*length1 + length1*length1)}" ixy="0.0" ixz="0.0"
+    iyy="${mass_palm / 12.0 * (length1*length1 + length1*length1)}" iyz="0.0"
+    izz="${mass_palm / 12.0 * (length1*length1 + length1*length1)}"/>
     </inertial>
   </link>
@@ -459,9 +559,9 @@
     <inertial>
       <origin xyz="${-x_width/2} 0 ${0.15/2}" rpy="0 0 0"/>
-      <mass value="${mass}"/>
-      <inertia
-    ixx="${mass / 12.0 * (width*width + width*width)}" ixy="0.0" ixz="0.0"
-    iyy="${mass / 12.0 * (length2*length2 + width*width)}" iyz="0.0"
-    izz="${mass / 12.0 * (width*width + length2*length2)}"/>
+      <mass value="${mass_palm}"/>
+      <inertia
+    ixx="${mass_palm / 12.0 * (width*width + width*width)}" ixy="0.0" ixz="0.0"
+    iyy="${mass_palm / 12.0 * (length2*length2 + width*width)}" iyz="0.0"
+    izz="${mass_palm / 12.0 * (width*width + length2*length2)}"/>
     </inertial>
   </link>
@@ -490,9 +590,9 @@
     <inertial>
       <origin xyz="${-x_width/2} 0 ${0.15/2}" rpy="0 0 0"/>
-      <mass value="${mass}"/>
-      <inertia
-    ixx="${mass / 12.0 * (width*width + width*width)}" ixy="0.0" ixz="0.0"
-    iyy="${mass / 12.0 * (length2*length2 + width*width)}" iyz="0.0"
-    izz="${mass / 12.0 * (width*width + length2*length2)}"/>
+      <mass value="${mass_palm}"/>
+      <inertia
+    ixx="${mass_palm / 12.0 * (width*width + width*width)}" ixy="0.0" ixz="0.0"
+    iyy="${mass_palm / 12.0 * (length2*length2 + width*width)}" iyz="0.0"
+    izz="${mass_palm / 12.0 * (width*width + length2*length2)}"/>
     </inertial>
   </link>
@@ -598,3 +698,43 @@
     </actuator>
   </transmission>
+  <transmission name="tran_Right_hinge">
+    <type>transmission_interface/SimpleTransmission</type>
+    <joint name="Right_hinge">
+      <hardwareInterface>hardware_interface/EffortJointInterface</hardwareInterface>
+    </joint>
+    <actuator name="motor_Right_hinge">
+      <hardwareInterface>hardware_interface/EffortJointInterface</hardwareInterface>
+      <mechanicalReduction>1</mechanicalReduction>
+    </actuator>
+  </transmission>
+  <transmission name="tran_Right_palm_x">
+    <type>transmission_interface/SimpleTransmission</type>
+    <joint name="Right_palm_x">
+      <hardwareInterface>hardware_interface/EffortJointInterface</hardwareInterface>
+    </joint>
+    <actuator name="motor_Right_palm_x">
+      <hardwareInterface>hardware_interface/EffortJointInterface</hardwareInterface>
+      <mechanicalReduction>1</mechanicalReduction>
+    </actuator>
+  </transmission>
+  <transmission name="tran_Right_palm_z">
+    <type>transmission_interface/SimpleTransmission</type>
+    <joint name="Right_palm_z">
+      <hardwareInterface>hardware_interface/EffortJointInterface</hardwareInterface>
+    </joint>
+    <actuator name="motor_Right_palm_z">
+      <hardwareInterface>hardware_interface/EffortJointInterface</hardwareInterface>
+      <mechanicalReduction>1</mechanicalReduction>
+    </actuator>
+  </transmission>
+  <transmission name="tran_Right_palm_y">
+    <type>transmission_interface/SimpleTransmission</type>
+    <joint name="Right_palm_y">
+      <hardwareInterface>hardware_interface/EffortJointInterface</hardwareInterface>
+    </joint>
+    <actuator name="motor_Right_palm_y">
+      <hardwareInterface>hardware_interface/EffortJointInterface</hardwareInterface>
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