Commit message: Fixed joints with just two movabel

File: src/baby/baby_description/urdf/baby.xacro (robot description, xacro)
@@ -8,5 +8,5 @@
   <xacro:property name="mass_neck" value="2" />
   <xacro:property name="mass_leg" value="25" />
-  <xacro:property name="mass_foot" value="10" />
+  <xacro:property name="mass_foot" value="1000" />
   <xacro:property name="radius" value="0.05" /> <!-- Radii of the cylinder-->
   <xacro:property name="length1" value="0.1" /> <!-- Right_seg42 -->
@@ -84,13 +84,13 @@
     <limit effort="1000.0" lower="0" upper="3.14" velocity="10"/>
   </joint>
-  <joint name="Neck_y_joint" type="revolute">
+  <joint name="Neck_y_joint" type="fixed">
     <parent link="Chest"/>
     <child link="Neck"/>
-    <origin xyz="0 0 ${chest_height}" rpy="0 -1.57 0"/>
+    <origin xyz="0 0 ${chest_height}" rpy="0 0 0"/>
     <axis xyz="0 1 0"/>
     <dynamics damping="0.7"/>
     <limit effort="1000.0" lower="0" upper="3.14" velocity="10"/>
   </joint>
-  <joint name="Left_leg_y" type="revolute">
+  <joint name="Left_leg_y" type="fixed">
     <parent link="Chest"/>
     <child link="Left_leg_upper"/>
@@ -100,5 +100,5 @@
     <limit effort="1000.0" lower="0" upper="3.14" velocity="10"/>
   </joint>
-  <joint name="Right_leg_y" type="revolute">
+  <joint name="Right_leg_y" type="fixed">
     <parent link="Chest"/>
     <child link="Right_leg_upper"/>
@@ -131,5 +131,5 @@
     </inertial>
   </link>
-  <joint name="Left_leg_hinge" type="revolute">
+  <joint name="Left_leg_hinge" type="fixed">
     <parent link="Left_leg_upper"/>
     <child link="Left_leg_lower"/>
@@ -161,5 +161,5 @@
     </inertial>
   </link>
-  <joint name="Left_foot_y" type="revolute">
+  <joint name="Left_foot_y" type="fixed">
     <parent link="Left_leg_lower"/>
     <child link="Left_foot"/>
@@ -214,5 +214,5 @@
     </inertial>
   </link>
-  <joint name="Right_leg_hinge" type="revolute">
+  <joint name="Right_leg_hinge" type="fixed">
     <parent link="Right_leg_upper"/>
     <child link="Right_leg_lower"/>
@@ -244,5 +244,5 @@
     </inertial>
   </link>
-  <joint name="Right_foot_y" type="revolute">
+  <joint name="Right_foot_y" type="fixed">
     <parent link="Right_leg_lower"/>
     <child link="Right_foot"/>
@@ -297,5 +297,5 @@
     </inertial>
   </link>
- <joint name="Head_z_joint" type="continuous">
+ <joint name="Head_z_joint" type="fixed">
     <parent link="Neck"/>
     <child link="Head_z"/>
@@ -326,8 +326,8 @@
     </inertial>
   </link>
-  <joint name="Head_x_joint" type="continuous">
+  <joint name="Head_x_joint" type="fixed">
     <parent link="Neck"/>
     <child link="Head"/>
-    <origin xyz="0 0 ${neck_height}" rpy="-1.57 0 0"/>
+    <origin xyz="0 0 ${neck_height}" rpy="0 0 0"/>
     <axis xyz="1 0 0"/>
     <limit effort="1000" velocity="1.0" />
@@ -378,5 +378,5 @@
     </inertial>
   </link>
-  <joint name="Right_hinge" type="revolute">
+  <joint name="Right_hinge" type="fixed">
     <parent link="Right_upper"/>
     <child link="Right_lower"/>
@@ -410,5 +410,5 @@
 <!-- ===============3 axis PALM joint =======================================
     ===== https://answers.ros.org/question/258420/ball-joint-in-urdf/  -->
-   <joint name="Right_palm_y" type="revolute">
+   <joint name="Right_palm_y" type="fixed">
     <parent link="Right_lower"/>
     <child link="Right_palm"/>
@@ -974,5 +974,5 @@
     </inertial>
   </link>
-  <joint name="Left_hinge" type="revolute">
+  <joint name="Left_hinge" type="fixed">
     <parent link="Left_upper"/>
     <child link="Left_lower"/>
@@ -1006,5 +1006,5 @@
 <!-- ===============3 axis PALM joint =======================================
     ===== https://answers.ros.org/question/258420/ball-joint-in-urdf/  -->
-   <joint name="Left_palm_y" type="revolute">
+   <joint name="Left_palm_y" type="fixed">
     <parent link="Left_lower"/>
     <child link="Left_palm"/>
@@ -1549,5 +1549,5 @@
 <!-- ==================TRANSMISSION LINE =========================== -->
 <!-- ============================= Head transmission ========================== -->
-  <transmission name="tran_Neck_y_joint">
+<!--   <transmission name="tran_Neck_y_joint">
     <type>transmission_interface/SimpleTransmission</type>
     <joint name="Neck_y_joint">
@@ -1579,6 +1579,7 @@
     </actuator>
   </transmission>
+ -->
 <!-- ============================= Leg transmission ========================== -->
-  <transmission name="tran_Right_leg_y">
+<!--   <transmission name="tran_Right_leg_y">
     <type>transmission_interface/SimpleTransmission</type>
     <joint name="Right_leg_y">
@@ -1639,16 +1640,69 @@
       <mechanicalReduction>1</mechanicalReduction>
     </actuator>
-  </transmission>
+  </transmission>-->
 <!-- ============================= Hand transmission ========================== -->
   <transmission name="tran_Right_hand_y">
     <type>transmission_interface/SimpleTransmission</type>
     <joint name="Right_hand_y">
-      <hardwareInterface>hardware_interface/PositionJointInterface</hardwareInterface>
+      <hardwareInterface>hardware_interface/EffortJointInterface</hardwareInterface>
     </joint>
     <actuator name="motor_Right_hand_y">
-      <hardwareInterface>hardware_interface/PositionJointInterface</hardwareInterface>
-      <mechanicalReduction>1</mechanicalReduction>
-    </actuator>
-  </transmission>
+      <hardwareInterface>hardware_interface/EffortJointInterface</hardwareInterface>
+      <mechanicalReduction>1</mechanicalReduction>
+    </actuator>
+  </transmission>
+  <transmission name="tran_Left_hand_y">
+    <type>transmission_interface/SimpleTransmission</type>
+    <joint name="Left_hand_y">
+      <hardwareInterface>hardware_interface/EffortJointInterface</hardwareInterface>
+    </joint>
+    <actuator name="motor_Left_hand_y">
+      <hardwareInterface>hardware_interface/EffortJointInterface</hardwareInterface>
+      <mechanicalReduction>1</mechanicalReduction>
+    </actuator>
+  </transmission>
+ <!--  <transmission name="tran_Right_hinge">
+    <type>transmission_interface/SimpleTransmission</type>
+    <joint name="Right_hinge">
+      <hardwareInterface>hardware_interface/PositionJointInterface</hardwareInterface>
+    </joint>
+    <actuator name="motor_Right_hinge">
+      <hardwareInterface>hardware_interface/PositionJointInterface</hardwareInterface>
+      <mechanicalReduction>1</mechanicalReduction>
+    </actuator>
+  </transmission>
+  <transmission name="tran_Right_palm_y">
+    <type>transmission_interface/SimpleTransmission</type>
+    <joint name="Right_palm_y">
+      <hardwareInterface>hardware_interface/PositionJointInterface</hardwareInterface>
+    </joint>
+    <actuator name="motor_Right_palm_y">
+      <hardwareInterface>hardware_interface/PositionJointInterface</hardwareInterface>
+      <mechanicalReduction>1</mechanicalReduction>
+    </actuator>
+  </transmission>
+ -->
+<!--   <transmission name="tran_Left_hinge">
+    <type>transmission_interface/SimpleTransmission</type>
+    <joint name="Left_hinge">
+      <hardwareInterface>hardware_interface/PositionJointInterface</hardwareInterface>
+    </joint>
+    <actuator name="motor_Left_hinge">
+      <hardwareInterface>hardware_interface/PositionJointInterface</hardwareInterface>
+      <mechanicalReduction>1</mechanicalReduction>
+    </actuator>
+  </transmission>
+  <transmission name="tran_Left_palm_y">
+    <type>transmission_interface/SimpleTransmission</type>
+    <joint name="Left_palm_y">
+      <hardwareInterface>hardware_interface/PositionJointInterface</hardwareInterface>
+    </joint>
+    <actuator name="motor_Left_palm_y">
+      <hardwareInterface>hardware_interface/PositionJointInterface</hardwareInterface>
+      <mechanicalReduction>1</mechanicalReduction>
+    </actuator>
+  </transmission>
+ -->
+<!--==========================Right palm ========================== -->
   <transmission name="Right_trant1">
     <type>transmission_interface/SimpleTransmission</type>
@@ -1751,35 +1805,5 @@
     </actuator>
   </transmission>
-  <transmission name="tran_Right_hinge">
-    <type>transmission_interface/SimpleTransmission</type>
-    <joint name="Right_hinge">
-      <hardwareInterface>hardware_interface/PositionJointInterface</hardwareInterface>
-    </joint>
-    <actuator name="motor_Right_hinge">
-      <hardwareInterface>hardware_interface/PositionJointInterface</hardwareInterface>
-      <mechanicalReduction>1</mechanicalReduction>
-    </actuator>
-  </transmission>
-  <transmission name="tran_Right_palm_y">
-    <type>transmission_interface/SimpleTransmission</type>
-    <joint name="Right_palm_y">
-      <hardwareInterface>hardware_interface/PositionJointInterface</hardwareInterface>
-    </joint>
-    <actuator name="motor_Right_palm_y">
-      <hardwareInterface>hardware_interface/PositionJointInterface</hardwareInterface>
-      <mechanicalReduction>1</mechanicalReduction>
-    </actuator>
-  </transmission>
-  <!-- Left hand transmissions -->
-  <transmission name="tran_Left_hand_y">
-    <type>transmission_interface/SimpleTransmission</type>
-    <joint name="Left_hand_y">
-      <hardwareInterface>hardware_interface/PositionJointInterface</hardwareInterface>
-    </joint>
-    <actuator name="motor_Left_hand_y">
-      <hardwareInterface>hardware_interface/PositionJointInterface</hardwareInterface>
-      <mechanicalReduction>1</mechanicalReduction>
-    </actuator>
-  </transmission>
+<!--================================= Left hand transmissions==================== -->
   <transmission name="Left_trant1">
     <type>transmission_interface/SimpleTransmission</type>
@@ -1878,24 +1902,4 @@
     </joint>
     <actuator name="Left_motor42">
-      <hardwareInterface>hardware_interface/PositionJointInterface</hardwareInterface>
-      <mechanicalReduction>1</mechanicalReduction>
-    </actuator>
-  </transmission>
-  <transmission name="tran_Left_hinge">
-    <type>transmission_interface/SimpleTransmission</type>
-    <joint name="Left_hinge">
-      <hardwareInterface>hardware_interface/PositionJointInterface</hardwareInterface>
-    </joint>
-    <actuator name="motor_Left_hinge">
-      <hardwareInterface>hardware_interface/PositionJointInterface</hardwareInterface>
-      <mechanicalReduction>1</mechanicalReduction>
-    </actuator>
-  </transmission>
-  <transmission name="tran_Left_palm_y">
-    <type>transmission_interface/SimpleTransmission</type>
-    <joint name="Left_palm_y">
-      <hardwareInterface>hardware_interface/PositionJointInterface</hardwareInterface>
-    </joint>
-    <actuator name="motor_Left_palm_y">
       <hardwareInterface>hardware_interface/PositionJointInterface</hardwareInterface>
       <mechanicalReduction>1</mechanicalReduction>
