Commit message: Major breakthrough in effort pid values.Mass remains a problem

File: src/baby/baby_description/urdf/baby.xacro (robot description, xacro)
@@ -4,37 +4,38 @@
   <xacro:property name="PI" value="3.1415926535897931"/>
   <xacro:property name="mass_chest" value="25" />
-  <xacro:property name="mass_palm" value="0.2" /> <!-- arbitrary value for mass -->
-  <xacro:property name="mass_hand" value="20" /> <!-- arbitrary value for mass -->
-  <xacro:property name="mass_neck" value="2" />
-  <xacro:property name="mass_leg" value="25" />
-  <xacro:property name="mass_foot" value="10" />
-  <xacro:property name="mass_dummy" value="0.2" />
+  <xacro:property name="mass_palm" value="00.2" /> <!-- arbitrary value for mass -->
+  <xacro:property name="mass_hand" value="05" /> <!-- arbitrary value for mass -->
+  <xacro:property name="mass_neck" value="02" />
+  <xacro:property name="mass_leg" value="10" />
+  <xacro:property name="mass_foot" value="5" />
+  <xacro:property name="mass_dummy" value="2.0" />
+  <!-- Total weight=0.2*8+5*2+10*4+2*1+6*1+5*4+0.2*32+25=1.6+10+40+2+6+20+6.4+25 -->
   <xacro:property name="radius" value="0.05" /> <!-- Radii of the cylinder-->
-  <xacro:property name="length1" value="0.1" /> <!-- Right_seg42 -->
-  <xacro:property name="length2" value="0.2" /> <!-- Rotator -->
-  <xacro:property name="width" value="0.1" /> <!-- width of the beam -->
-  <xacro:property name="imr_width" value="0.173" /> <!-- index middle ring finger width -->
-  <xacro:property name="l_width" value="0.15" /> <!-- little finger width -->
-  <xacro:property name="x_width" value="0.10" />
-  <xacro:property name="hand_height" value="2" /> <!-- little width -->
-  <xacro:property name="hand_radius" value="0.20" /> <!-- little width -->
-  <xacro:property name="chest_height" value="6" /><!-- z-->
-  <xacro:property name="chest_width" value="0.5" /><!-- x-->
-  <xacro:property name="chest_length" value="3" /><!--y-->
-  <xacro:property name="palm_height" value="1.1" />
-  <xacro:property name="palm_length" value="1" /><!--y-->
-  <xacro:property name="palm_width" value="0.3" /><!--x-->
+  <xacro:property name="length1" value="0.01" /> <!-- Right_seg42 -->
+  <xacro:property name="length2" value="0.02" /> <!-- Rotator -->
+  <xacro:property name="width" value="0.01" /> <!-- width of the beam -->
+  <xacro:property name="imr_width" value="0.0173" /> <!-- index middle ring finger width -->
+  <xacro:property name="l_width" value="0.015" /> <!-- little finger width -->
+  <xacro:property name="x_width" value="0.010" />
+  <xacro:property name="hand_height" value="0.2" /> <!-- little width -->
+  <xacro:property name="hand_radius" value="0.020" /> <!-- little width -->
+  <xacro:property name="chest_height" value="0.6" /><!-- z-->
+  <xacro:property name="chest_width" value="0.05" /><!-- x-->
+  <xacro:property name="chest_length" value="0.3" /><!--y-->
+  <xacro:property name="palm_height" value="0.11" />
+  <xacro:property name="palm_length" value="0.1" /><!--y-->
+  <xacro:property name="palm_width" value="0.03" /><!--x-->
   <xacro:property name="spacing" value="${(palm_length-imr_width/2-l_width/2)/3}" />
-  <xacro:property name="neck_height" value="0.4" />
-  <xacro:property name="neck_radius" value="0.2" />
-  <xacro:property name="head_height" value="0.8" />
-  <xacro:property name="head_radius" value="0.5" />
-  <xacro:property name="leg_height" value="2" />
-  <xacro:property name="leg_radius" value="0.2" />
-  <xacro:property name="foot_height" value="0.2" />
-  <xacro:property name="foot_length" value="1" />
-  <xacro:property name="foot_width" value="1" />
-  <xacro:property name="dummy_size" value="1.0" />
-  <xacro:property name="dummy_size_leg" value="2.0" />
+  <xacro:property name="neck_height" value="0.04" />
+  <xacro:property name="neck_radius" value="0.02" />
+  <xacro:property name="head_height" value="0.08" />
+  <xacro:property name="head_radius" value="0.05" />
+  <xacro:property name="leg_height" value="0.2" />
+  <xacro:property name="leg_radius" value="0.02" />
+  <xacro:property name="foot_height" value="0.02" />
+  <xacro:property name="foot_length" value="0.1" />
+  <xacro:property name="foot_width" value="0.1" />
+  <xacro:property name="dummy_size" value="0.10" />
+  <xacro:property name="dummy_size_leg" value="0.20" />
   <xacro:include filename="$(find baby_description)/urdf/baby.gazebo" />
   <xacro:include filename="$(find baby_description)/urdf/materials.xacro" />
@@ -91,8 +92,8 @@
     <parent link="Chest"/>
     <child link="Neck"/>
-    <origin xyz="0 0 ${chest_height}" rpy="0 -1.57 0"/>
-    <axis xyz="0 1 0"/>
-    <dynamics damping="0.7"/>
-    <limit effort="1000.0" lower="0" upper="3.14" velocity="10"/>
+    <origin xyz="0 0 ${chest_height}" rpy="0 0 0"/>
+    <axis xyz="0 1 0"/>
+    <dynamics damping="0.7"/>
+    <limit effort="1000.0" lower="-1.57" upper="1.57" velocity="10"/>
   </joint>
   <joint name="Left_leg_y" type="revolute">
@@ -407,5 +408,5 @@
     <parent link="Neck"/>
     <child link="Head"/>
-    <origin xyz="0 0 ${neck_height}" rpy="-1.57 0 0"/>
+    <origin xyz="0 0 ${neck_height}" rpy="0 0 0"/>
     <axis xyz="1 0 0"/>
     <limit effort="1000" velocity="1.0" />
@@ -619,18 +620,18 @@
   <link name="Right_segt1">
     <collision>
-      <origin xyz="0 0 ${0.15/2}" rpy="0 0 0"/>
-      <geometry>
-         <box size="${x_width} 0.21 0.15"/>
-      </geometry>
-    </collision>
-    <visual>
-      <origin xyz="0 0 ${0.15/2}" rpy="0 0 0"/>
-      <geometry>
-         <box size="${x_width} 0.21 0.15"/>
+      <origin xyz="0 0 ${0.015/2}" rpy="0 0 0"/>
+      <geometry>
+         <box size="${x_width} 0.021 0.015"/>
+      </geometry>
+    </collision>
+    <visual>
+      <origin xyz="0 0 ${0.015/2}" rpy="0 0 0"/>
+      <geometry>
+         <box size="${x_width} 0.021 0.015"/>
       </geometry>
       <material name="orange"/>
     </visual>
     <inertial>
-      <origin xyz="0 0 ${0.15/2}" rpy="0 0 0"/>
+      <origin xyz="0 0 ${0.015/2}" rpy="0 0 0"/>
       <mass value="${mass_palm}"/>
       <inertia
@@ -643,5 +644,5 @@
     <parent link="Right_segt1"/>
     <child link="Right_segt2"/>
-    <origin xyz="${x_width/2} 0 0.15" rpy="0 0 0"/>
+    <origin xyz="${x_width/2} 0 0.015" rpy="0 0 0"/>
     <axis xyz="0 1 0"/>
     <dynamics damping="0.7"/>
@@ -650,18 +651,18 @@
   <link name="Right_segt2">
     <collision>
-      <origin xyz="${-x_width/2} 0 ${0.268/2}" rpy="0 0 0"/>
-      <geometry>
-         <box size="${x_width} 0.21 0.268"/>
-      </geometry>
-    </collision>
-    <visual>
-      <origin xyz="${-x_width/2} 0 ${0.268/2}" rpy="0 0 0"/>
-      <geometry>
-         <box size="${x_width} 0.21 0.268"/>
+      <origin xyz="${-x_width/2} 0 ${0.0268/2}" rpy="0 0 0"/>
+      <geometry>
+         <box size="${x_width} 0.021 0.0268"/>
+      </geometry>
+    </collision>
+    <visual>
+      <origin xyz="${-x_width/2} 0 ${0.0268/2}" rpy="0 0 0"/>
+      <geometry>
+         <box size="${x_width} 0.021 0.0268"/>
       </geometry>
       <material name="black"/>
     </visual>
     <inertial>
-      <origin xyz="${-x_width/2} 0 ${0.268/2}" rpy="0 0 0"/>
+      <origin xyz="${-x_width/2} 0 ${0.0268/2}" rpy="0 0 0"/>
       <mass value="${mass_palm}"/>
       <inertia
@@ -674,5 +675,5 @@
     <parent link="Right_segt2"/>
     <child link="Right_segt3"/>
-    <origin xyz="0 0 ${0.268}" rpy="0 0 0"/>
+    <origin xyz="0 0 ${0.0268}" rpy="0 0 0"/>
     <axis xyz="0 1 0"/>
     <dynamics damping="0.7"/>
@@ -681,18 +682,18 @@
   <link name="Right_segt3">
     <collision>
-      <origin xyz="${-x_width/2} 0 ${0.268/2}" rpy="0 0 0"/>
-      <geometry>
-         <box size="${x_width} 0.21 0.268"/>
-      </geometry>
-    </collision>
-    <visual>
-      <origin xyz="${-x_width/2} 0 ${0.268/2}" rpy="0 0 0"/>
-      <geometry>
-         <box size="${x_width} 0.21 0.268"/>
+      <origin xyz="${-x_width/2} 0 ${0.0268/2}" rpy="0 0 0"/>
+      <geometry>
+         <box size="${x_width} 0.021 0.0268"/>
+      </geometry>
+    </collision>
+    <visual>
+      <origin xyz="${-x_width/2} 0 ${0.0268/2}" rpy="0 0 0"/>
+      <geometry>
+         <box size="${x_width} 0.021 0.0268"/>
       </geometry>
       <material name="black"/>
     </visual>
     <inertial>
-      <origin xyz="${-x_width/2} 0 ${0.268/2}" rpy="0 0 0"/>
+      <origin xyz="${-x_width/2} 0 ${0.0268/2}" rpy="0 0 0"/>
       <mass value="${mass_palm}"/>
       <inertia
@@ -705,18 +706,18 @@
   <link name="Right_seg11">
     <collision>
-      <origin xyz="0 0 ${0.268/2}" rpy="0 0 0"/>
-      <geometry>
-	       <box size="${x_width} ${imr_width} 0.268"/>
-      </geometry>
-    </collision>
-    <visual>
-      <origin xyz="0 0 ${0.268/2}" rpy="0 0 0"/>
-      <geometry>
-	       <box size="${x_width} ${imr_width} 0.268"/>
+      <origin xyz="0 0 ${0.0268/2}" rpy="0 0 0"/>
+      <geometry>
+	       <box size="${x_width} ${imr_width} 0.0268"/>
+      </geometry>
+    </collision>
+    <visual>
+      <origin xyz="0 0 ${0.0268/2}" rpy="0 0 0"/>
+      <geometry>
+	       <box size="${x_width} ${imr_width} 0.0268"/>
       </geometry>
       <material name="orange"/>
     </visual>
     <inertial>
-      <origin xyz="0 0 ${0.268/2}" rpy="0 0 0"/>
+      <origin xyz="0 0 ${0.0268/2}" rpy="0 0 0"/>
       <mass value="${mass_palm}"/>
       <inertia
@@ -729,5 +730,5 @@
     <parent link="Right_seg11"/>
     <child link="Right_seg12"/>
-    <origin xyz="${x_width/2} 0 0.268" rpy="0 0 0"/>
+    <origin xyz="${x_width/2} 0 0.0268" rpy="0 0 0"/>
     <axis xyz="0 1 0"/>
     <dynamics damping="0.7"/>
@@ -736,18 +737,18 @@
   <link name="Right_seg12">
     <collision>
-      <origin xyz="${-x_width/2} 0 ${0.268/2}" rpy="0 0 0"/>
-      <geometry>
-	       <box size="${x_width} ${imr_width} 0.268"/>
-      </geometry>
-    </collision>
-    <visual>
-      <origin xyz="${-x_width/2} 0 ${0.268/2}" rpy="0 0 0"/>
-      <geometry>
-	       <box size="${x_width} ${imr_width} 0.268"/>
+      <origin xyz="${-x_width/2} 0 ${0.0268/2}" rpy="0 0 0"/>
+      <geometry>
+	       <box size="${x_width} ${imr_width} 0.0268"/>
+      </geometry>
+    </collision>
+    <visual>
+      <origin xyz="${-x_width/2} 0 ${0.0268/2}" rpy="0 0 0"/>
+      <geometry>
+	       <box size="${x_width} ${imr_width} 0.0268"/>
       </geometry>
       <material name="black"/>
     </visual>
     <inertial>
-      <origin xyz="${-x_width/2} 0 ${0.268/2}" rpy="0 0 0"/>
+      <origin xyz="${-x_width/2} 0 ${0.0268/2}" rpy="0 0 0"/>
       <mass value="${mass_palm}"/>
       <inertia
@@ -760,5 +761,5 @@
     <parent link="Right_seg12"/>
     <child link="Right_seg13"/>
-    <origin xyz="0 0 ${0.268}" rpy="0 0 0"/>
+    <origin xyz="0 0 ${0.0268}" rpy="0 0 0"/>
     <axis xyz="0 1 0"/>
     <dynamics damping="0.7"/>
@@ -767,18 +768,18 @@
   <link name="Right_seg13">
     <collision>
-      <origin xyz="${-x_width/2} 0 ${0.268/2}" rpy="0 0 0"/>
-      <geometry>
-         <box size="${x_width} ${imr_width} 0.268"/>
-      </geometry>
-    </collision>
-    <visual>
-      <origin xyz="${-x_width/2} 0 ${0.268/2}" rpy="0 0 0"/>
-      <geometry>
-         <box size="${x_width} ${imr_width} 0.268"/>
+      <origin xyz="${-x_width/2} 0 ${0.0268/2}" rpy="0 0 0"/>
+      <geometry>
+         <box size="${x_width} ${imr_width} 0.0268"/>
+      </geometry>
+    </collision>
+    <visual>
+      <origin xyz="${-x_width/2} 0 ${0.0268/2}" rpy="0 0 0"/>
+      <geometry>
+         <box size="${x_width} ${imr_width} 0.0268"/>
       </geometry>
       <material name="black"/>
     </visual>
     <inertial>
-      <origin xyz="${-x_width/2} 0 ${0.268/2}" rpy="0 0 0"/>
+      <origin xyz="${-x_width/2} 0 ${0.0268/2}" rpy="0 0 0"/>
       <mass value="${mass_palm}"/>
       <inertia
@@ -791,5 +792,5 @@
   <link name="Right_seg21">
     <collision>
-      <origin xyz="0 0 ${0.3/2}" rpy="0 0 0"/>
+      <origin xyz="0 0 ${0.03/2}" rpy="0 0 0"/>
       <geometry>
          <box size="${x_width} ${imr_width} 0.2"/>
@@ -797,12 +798,12 @@
     </collision>
     <visual>
-      <origin xyz="0 0 ${0.3/2}" rpy="0 0 0"/>
-      <geometry>
-         <box size="${x_width} ${imr_width} 0.3"/>
+      <origin xyz="0 0 ${0.03/2}" rpy="0 0 0"/>
+      <geometry>
+         <box size="${x_width} ${imr_width} 0.03"/>
       </geometry>
       <material name="orange"/>
     </visual>
     <inertial>
-      <origin xyz="0 0 ${0.3/2}" rpy="0 0 0"/>
+      <origin xyz="0 0 ${0.03/2}" rpy="0 0 0"/>
       <mass value="${mass_palm}"/>
       <inertia
@@ -815,5 +816,5 @@
     <parent link="Right_seg21"/>
     <child link="Right_seg22"/>
-    <origin xyz="${x_width/2} 0.0 0.3" rpy="0 0 0"/>
+    <origin xyz="${x_width/2} 0.0 0.03" rpy="0 0 0"/>
     <axis xyz="0 1 0"/>
     <dynamics damping="0.7"/>
@@ -822,18 +823,18 @@
   <link name="Right_seg22">
     <collision>
-      <origin xyz="${-x_width/2} 0 ${0.3/2}" rpy="0 0 0"/>
-      <geometry>
-         <box size="${x_width} ${imr_width} 0.3"/>
-      </geometry>
-    </collision>
-    <visual>
-      <origin xyz="${-x_width/2} 0 ${0.3/2}" rpy="0 0 0"/>
-      <geometry>
-         <box size="${x_width} ${imr_width} 0.3"/>
+      <origin xyz="${-x_width/2} 0 ${0.03/2}" rpy="0 0 0"/>
+      <geometry>
+         <box size="${x_width} ${imr_width} 0.03"/>
+      </geometry>
+    </collision>
+    <visual>
+      <origin xyz="${-x_width/2} 0 ${0.03/2}" rpy="0 0 0"/>
+      <geometry>
+         <box size="${x_width} ${imr_width} 0.03"/>
       </geometry>
       <material name="black"/>
     </visual>
     <inertial>
-      <origin xyz="${-x_width/2} 0 ${0.3/2}" rpy="0 0 0"/>
+      <origin xyz="${-x_width/2} 0 ${0.03/2}" rpy="0 0 0"/>
       <mass value="${mass_palm}"/>
       <inertia
@@ -846,5 +847,5 @@
     <parent link="Right_seg22"/>
     <child link="Right_seg23"/>
-    <origin xyz="0 0 0.3" rpy="0 0 0"/>
+    <origin xyz="0 0 0.03" rpy="0 0 0"/>
     <axis xyz="0 1 0"/>
     <dynamics damping="0.7"/>
@@ -853,18 +854,18 @@
   <link name="Right_seg23">
     <collision>
-      <origin xyz="${-x_width/2} 0 ${0.3/2}" rpy="0 0 0"/>
-      <geometry>
-         <box size="${x_width} ${imr_width} 0.3"/>
-      </geometry>
-    </collision>
-    <visual>
-      <origin xyz="${-x_width/2} 0 ${0.3/2}" rpy="0 0 0"/>
-      <geometry>
-         <box size="${x_width} ${imr_width} 0.3"/>
+      <origin xyz="${-x_width/2} 0 ${0.03/2}" rpy="0 0 0"/>
+      <geometry>
+         <box size="${x_width} ${imr_width} 0.03"/>
+      </geometry>
+    </collision>
+    <visual>
+      <origin xyz="${-x_width/2} 0 ${0.03/2}" rpy="0 0 0"/>
+      <geometry>
+         <box size="${x_width} ${imr_width} 0.03"/>
       </geometry>
       <material name="black"/>
     </visual>
     <inertial>
-      <origin xyz="${-x_width/2} 0 ${0.3/2}" rpy="0 0 0"/>
+      <origin xyz="${-x_width/2} 0 ${0.03/2}" rpy="0 0 0"/>
       <mass value="${mass_palm}"/>
       <inertia
@@ -877,18 +878,18 @@
   <link name="Right_seg31">
     <collision>
-      <origin xyz="0 0 ${0.24/2}" rpy="0 0 0"/>
-      <geometry>
-         <box size="${x_width} ${imr_width} 0.24"/>
-      </geometry>
-    </collision>
-    <visual>
-      <origin xyz="0 0 ${0.24/2}" rpy="0 0 0"/>
-      <geometry>
-         <box size="${x_width} ${imr_width} 0.24"/>
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
Commit message: Modified the parameters

File: src/baby/baby_description/urdf/baby.xacro (robot description, xacro)
@@ -4,9 +4,9 @@
   <xacro:property name="PI" value="3.1415926535897931"/>
   <xacro:property name="mass_chest" value="25" />
-  <xacro:property name="mass_palm" value="00.2" /> <!-- arbitrary value for mass -->
+  <xacro:property name="mass_palm" value="0.2" /> <!-- arbitrary value for mass -->
   <xacro:property name="mass_hand" value="05" /> <!-- arbitrary value for mass -->
   <xacro:property name="mass_neck" value="02" />
   <xacro:property name="mass_leg" value="10" />
-  <xacro:property name="mass_foot" value="5" />
+  <xacro:property name="mass_foot" value="500" />
   <xacro:property name="mass_dummy" value="2.0" />
   <!-- Total weight=0.2*8+5*2+10*4+2*1+6*1+5*4+0.2*32+25=1.6+10+40+2+6+20+6.4+25 -->
@@ -48,5 +48,5 @@
     <limit effort="1000.0" lower="0" upper="6.20" velocity="10"/>
   </joint>
-<!--=======================Chest ========================================= -->
+<!--======================= Chest ========================================= -->
   <link name="Chest">
     <collision>
