Commit message: Added Walking files, hand movement, effort controllers, made base wider

File: src/baby/baby_description/urdf/baby.xacro (robot description, xacro)
@@ -3,18 +3,11 @@
   <!-- Constants for robot dimensions -->
   <xacro:property name="PI" value="3.1415926535897931"/>
-  <xacro:property name="mass_chest" value="25" />
+  <xacro:property name="mass_chest" value="30" />
   <xacro:property name="mass_palm" value="0.2" /> <!-- arbitrary value for mass -->
-<<<<<<< HEAD
-  <xacro:property name="mass_hand" value="20" /> <!-- arbitrary value for mass -->
-  <xacro:property name="mass_neck" value="2" />
-  <xacro:property name="mass_leg" value="25" />
-  <xacro:property name="mass_foot" value="1000" />
-=======
   <xacro:property name="mass_hand" value="05" /> <!-- arbitrary value for mass -->
   <xacro:property name="mass_neck" value="02" />
   <xacro:property name="mass_leg" value="10" />
-  <xacro:property name="mass_foot" value="500" />
+  <xacro:property name="mass_foot" value="5" />
   <xacro:property name="mass_dummy" value="2.0" />
->>>>>>> a1be921752e1b1a103237c6e8eefa59f6623a261
   <!-- Total weight=0.2*8+5*2+10*4+2*1+6*1+5*4+0.2*32+25=1.6+10+40+2+6+20+6.4+25 -->
   <xacro:property name="radius" value="0.05" /> <!-- Radii of the cylinder-->
@@ -22,7 +15,4 @@
   <xacro:property name="length2" value="0.02" /> <!-- Rotator -->
   <xacro:property name="width" value="0.01" /> <!-- width of the beam -->
-  <xacro:property name="imr_width" value="0.0173" /> <!-- index middle ring finger width -->
-  <xacro:property name="l_width" value="0.015" /> <!-- little finger width -->
-  <xacro:property name="x_width" value="0.010" />
   <xacro:property name="hand_height" value="0.2" /> <!-- little width -->
   <xacro:property name="hand_radius" value="0.020" /> <!-- little width -->
@@ -31,6 +21,14 @@
   <xacro:property name="chest_length" value="0.3" /><!--y-->
   <xacro:property name="palm_height" value="0.11" />
-  <xacro:property name="palm_length" value="0.1" /><!--y-->
-  <xacro:property name="palm_width" value="0.03" /><!--x-->
+  <xacro:property name="palm_length" value="0.1" /> <!--y-->
+  <xacro:property name="palm_width" value="0.03" /> <!--x-->
+  <xacro:property name="imr_width" value="0.0173" /> <!-- index middle ring finger width -->
+  <xacro:property name="l_width" value="0.015" /> <!-- little finger width -->
+  <xacro:property name="x_width" value="0.010" />
+  <xacro:property name="thulittle_height" value="0.015" /><!-- thumb and little finger height -->
+  <xacro:property name="thuind_height" value="0.0268" /><!-- thumb and index finger height -->
+  <xacro:property name="thumb_width" value="0.021" />
+  <xacro:property name="middle_height" value="0.03" />
+  <xacro:property name="ring_height" value="0.024" />
   <xacro:property name="spacing" value="${(palm_length-imr_width/2-l_width/2)/3}" />
   <xacro:property name="neck_height" value="0.04" />
@@ -41,6 +39,6 @@
   <xacro:property name="leg_radius" value="0.02" />
   <xacro:property name="foot_height" value="0.02" />
-  <xacro:property name="foot_length" value="0.1" />
-  <xacro:property name="foot_width" value="0.1" />
+  <xacro:property name="foot_length" value="0.4" />
+  <xacro:property name="foot_width" value="0.4" />
   <xacro:property name="dummy_size" value="0.10" />
   <xacro:property name="dummy_size_leg" value="0.20" />
@@ -83,5 +81,5 @@
     <parent link="Chest"/>
     <child link="Right_z_handD"/>
-    <origin xyz="0 ${chest_length/2} ${2*chest_height/3}" rpy="0 0 0"/>
+    <origin xyz="0 ${chest_length/2} ${chest_height}" rpy="0 0 0"/>
     <axis xyz="0 1 0"/>
     <dynamics damping="0.7"/>
@@ -91,10 +89,10 @@
     <parent link="Chest"/>
     <child link="Left_z_handD"/>
-    <origin xyz="0 ${-chest_length/2} ${2*chest_height/3}" rpy="0 0 0"/>
+    <origin xyz="0 ${-chest_length/2} ${chest_height}" rpy="0 0 0"/>
     <axis xyz="0 1 0"/>
     <dynamics damping="0.7"/>
     <limit effort="1000.0" lower="0" upper="6.20" velocity="10"/>
   </joint>
-  <joint name="Neck_y_joint" type="fixed">
+  <joint name="Neck_y_joint" type="revolute">
     <parent link="Chest"/>
     <child link="Neck"/>
@@ -104,5 +102,5 @@
     <limit effort="1000.0" lower="-1.57" upper="1.57" velocity="10"/>
   </joint>
-  <joint name="Left_leg_y" type="fixed">
+  <joint name="Left_leg_y" type="revolute">
     <parent link="Chest"/>
     <child link="Left_leg_upper"/>
@@ -110,7 +108,7 @@
     <axis xyz="0 1 0"/>
     <dynamics damping="0.7"/>
-    <limit effort="1000.0" lower="0" upper="3.14" velocity="10"/>
-  </joint>
-  <joint name="Right_leg_y" type="fixed">
+    <limit effort="1000.0" lower="-1.57" upper="1.57" velocity="10"/>
+  </joint>
+  <joint name="Right_leg_y" type="revolute">
     <parent link="Chest"/>
     <child link="Right_leg_upper"/>
@@ -118,5 +116,5 @@
     <axis xyz="0 1 0"/>
     <dynamics damping="0.7"/>
-    <limit effort="1000.0" lower="0" upper="3.14" velocity="10"/>
+    <limit effort="1000.0" lower="-1.57" upper="1.57" velocity="10"/>
   </joint>
 <!-- ========================3 axis leg joints ========================-->
@@ -217,5 +215,5 @@
     </inertial>
   </link>
-  <joint name="Left_leg_hinge" type="fixed">
+  <joint name="Left_leg_hinge" type="revolute">
     <parent link="Left_leg_upper"/>
     <child link="Left_leg_lower"/>
@@ -247,5 +245,5 @@
     </inertial>
   </link>
-  <joint name="Left_foot_y" type="fixed">
+  <joint name="Left_foot_y" type="revolute">
     <parent link="Left_leg_lower"/>
     <child link="Left_foot"/>
@@ -253,5 +251,5 @@
     <axis xyz="0 1 0"/>
     <dynamics damping="0.7"/>
-    <limit effort="1000.0" lower="0" upper="3.14" velocity="10"/>
+    <limit effort="1000.0" lower="-1.57" upper="1.57" velocity="10"/>
   </joint>
   <link name="Left_foot">
@@ -300,5 +298,5 @@
     </inertial>
   </link>
-  <joint name="Right_leg_hinge" type="fixed">
+  <joint name="Right_leg_hinge" type="revolute">
     <parent link="Right_leg_upper"/>
     <child link="Right_leg_lower"/>
@@ -330,5 +328,5 @@
     </inertial>
   </link>
-  <joint name="Right_foot_y" type="fixed">
+  <joint name="Right_foot_y" type="revolute">
     <parent link="Right_leg_lower"/>
     <child link="Right_foot"/>
@@ -336,5 +334,5 @@
     <axis xyz="0 1 0"/>
     <dynamics damping="0.7"/>
-    <limit effort="1000.0" lower="0" upper="3.14" velocity="10"/>
+    <limit effort="1000.0" lower="-1.57" upper="1.57" velocity="10"/>
   </joint>
   <link name="Right_foot">
@@ -383,5 +381,5 @@
     </inertial>
   </link>
- <joint name="Head_z_joint" type="fixed">
+ <joint name="Head_z_joint" type="revolute">
     <parent link="Neck"/>
     <child link="Head_z"/>
@@ -412,5 +410,5 @@
     </inertial>
   </link>
-  <joint name="Head_x_joint" type="fixed">
+  <joint name="Head_x_joint" type="revolute">
     <parent link="Neck"/>
     <child link="Head"/>
@@ -501,5 +499,5 @@
     </inertial>
   </link>
-  <joint name="Right_hinge" type="fixed">
+  <joint name="Right_hinge" type="revolute">
     <parent link="Right_upper"/>
     <child link="Right_lower"/>
@@ -533,5 +531,5 @@
 <!-- ===============3 axis PALM joint =======================================
     ===== https://answers.ros.org/question/258420/ball-joint-in-urdf/  -->
-   <joint name="Right_palm_y" type="fixed">
+   <joint name="Right_palm_y" type="revolute">
     <parent link="Right_lower"/>
     <child link="Right_x_palmD"/>
@@ -627,18 +625,190 @@
   <link name="Right_segt1">
     <collision>
-      <origin xyz="0 0 ${0.015/2}" rpy="0 0 0"/>
-      <geometry>
-         <box size="${x_width} 0.021 0.015"/>
-      </geometry>
-    </collision>
-    <visual>
-      <origin xyz="0 0 ${0.015/2}" rpy="0 0 0"/>
-      <geometry>
-         <box size="${x_width} 0.021 0.015"/>
+      <origin xyz="0 0 ${thulittle_height/2}" rpy="0 0 0"/>
+      <geometry>
+         <box size="${x_width} ${thumb_width} ${thulittle_height}"/>
+      </geometry>
+    </collision>
+    <visual>
+      <origin xyz="0 0 ${thulittle_height/2}" rpy="0 0 0"/>
+      <geometry>
+         <box size="${x_width} ${thumb_width} ${thulittle_height}"/>
       </geometry>
       <material name="orange"/>
     </visual>
     <inertial>
-      <origin xyz="0 0 ${0.015/2}" rpy="0 0 0"/>
+      <origin xyz="0 0 ${thulittle_height/2}" rpy="0 0 0"/>
+      <mass value="${mass_palm}"/>
+      <inertia
+    ixx="${mass_palm / 12.0 * (thumb_width*thumb_width + thulittle_height*thulittle_height)}" ixy="0.0" ixz="0.0"
+    iyy="${mass_palm / 12.0 * (thulittle_height*thulittle_height + x_width*x_width)}" iyz="0.0"
+    izz="${mass_palm / 12.0 * (x_width*x_width + thumb_width*thumb_width)}"/>
+    </inertial>
+  </link>
+  <joint name="Right_jointt1" type="revolute">
+    <parent link="Right_segt1"/>
+    <child link="Right_segt2"/>
+    <origin xyz="${x_width/2} 0 ${thulittle_height}" rpy="0 0 0"/>
+    <axis xyz="0 1 0"/>
+    <dynamics damping="0.7"/>
+    <limit effort="1000.0" lower="0" upper="1.57" velocity="10"/>
+  </joint>
+  <link name="Right_segt2">
+    <collision>
+      <origin xyz="${-x_width/2} 0 ${thuind_height/2}" rpy="0 0 0"/>
+      <geometry>
+         <box size="${x_width} ${thumb_width} ${thuind_height}"/>
+      </geometry>
+    </collision>
+    <visual>
+      <origin xyz="${-x_width/2} 0 ${thuind_height/2}" rpy="0 0 0"/>
+      <geometry>
+         <box size="${x_width} ${thumb_width} ${thuind_height}"/>
+      </geometry>
+      <material name="black"/>
+    </visual>
+    <inertial>
+      <origin xyz="${-x_width/2} 0 ${thuind_height/2}" rpy="0 0 0"/>
+      <mass value="${mass_palm}"/>
+      <inertia
+    ixx="${mass_palm / 12.0 * (thumb_width*thumb_width + thuind_height*thuind_height)}" ixy="0.0" ixz="0.0"
+    iyy="${mass_palm / 12.0 * (thuind_height*thuind_height + x_width*x_width)}" iyz="0.0"
+    izz="${mass_palm / 12.0 * (x_width*x_width + thumb_width*thumb_width)}"/>
+    </inertial>
+  </link>
+  <joint name="Right_jointt2" type="revolute">
+    <parent link="Right_segt2"/>
+    <child link="Right_segt3"/>
+    <origin xyz="0 0 ${thuind_height}" rpy="0 0 0"/>
+    <axis xyz="0 1 0"/>
+    <dynamics damping="0.7"/>
+    <limit effort="1000.0" lower="0" upper="1.57" velocity="10"/>
+  </joint>
+  <link name="Right_segt3">
+    <collision>
+      <origin xyz="${-x_width/2} 0 ${thuind_height/2}" rpy="0 0 0"/>
+      <geometry>
+         <box size="${x_width} ${thumb_width} ${thuind_height}"/>
+      </geometry>
+    </collision>
+    <visual>
+      <origin xyz="${-x_width/2} 0 ${thuind_height/2}" rpy="0 0 0"/>
+      <geometry>
+         <box size="${x_width} ${thumb_width} ${thuind_height}"/>
+      </geometry>
+      <material name="black"/>
+    </visual>
+    <inertial>
+      <origin xyz="${-x_width/2} 0 ${thuind_height/2}" rpy="0 0 0"/>
+      <mass value="${mass_palm}"/>
+      <inertia
+    ixx="${mass_palm / 12.0 * (thumb_width*thumb_width + thuind_height*thuind_height)}" ixy="0.0" ixz="0.0"
+    iyy="${mass_palm / 12.0 * (thuind_height*thuind_height + x_width*x_width)}" iyz="0.0"
+    izz="${mass_palm / 12.0 * (x_width*x_width + thumb_width*thumb_width)}"/>
+    </inertial>
+  </link>
+<!--====================== INDEX FINGER ===============================-->
+  <link name="Right_seg11">
+    <collision>
+      <origin xyz="0 0 ${thuind_height/2}" rpy="0 0 0"/>
+      <geometry>
+	       <box size="${x_width} ${imr_width} ${thuind_height}"/>
+      </geometry>
+    </collision>
+    <visual>
+      <origin xyz="0 0 ${thuind_height/2}" rpy="0 0 0"/>
+      <geometry>
+	       <box size="${x_width} ${imr_width} ${thuind_height}"/>
+      </geometry>
+      <material name="orange"/>
+    </visual>
+    <inertial>
+      <origin xyz="0 0 ${thuind_height/2}" rpy="0 0 0"/>
+      <mass value="${mass_palm}"/>
+      <inertia
+	  ixx="${mass_palm / 12.0 * (length1*length1 + length1*length1)}" ixy="0.0" ixz="0.0"
+	  iyy="${mass_palm / 12.0 * (length1*length1 + length1*length1)}" iyz="0.0"
+	  izz="${mass_palm / 12.0 * (length1*length1 + length1*length1)}"/>
+    </inertial>
+  </link>
+  <joint name="Right_joint11" type="revolute">
+    <parent link="Right_seg11"/>
+    <child link="Right_seg12"/>
+    <origin xyz="${x_width/2} 0 ${thuind_height}" rpy="0 0 0"/>
+    <axis xyz="0 1 0"/>
+    <dynamics damping="0.7"/>
+    <limit effort="1000.0" lower="0" upper="1.57" velocity="10"/>
+  </joint>
+  <link name="Right_seg12">
+    <collision>
+      <origin xyz="${-x_width/2} 0 ${thuind_height/2}" rpy="0 0 0"/>
+      <geometry>
+	       <box size="${x_width} ${imr_width} ${thuind_height}"/>
+      </geometry>
+    </collision>
+    <visual>
+      <origin xyz="${-x_width/2} 0 ${thuind_height/2}" rpy="0 0 0"/>
+      <geometry>
+	       <box size="${x_width} ${imr_width} ${thuind_height}"/>
+      </geometry>
+      <material name="black"/>
+    </visual>
+    <inertial>
+      <origin xyz="${-x_width/2} 0 ${thuind_height/2}" rpy="0 0 0"/>
+      <mass value="${mass_palm}"/>
+      <inertia
+	  ixx="${mass_palm / 12.0 * (width*width + width*width)}" ixy="0.0" ixz="0.0"
+	  iyy="${mass_palm / 12.0 * (length2*length2 + width*width)}" iyz="0.0"
+	  izz="${mass_palm / 12.0 * (width*width + length2*length2)}"/>
+    </inertial>
+  </link>
+  <joint name="Right_joint12" type="revolute">
+    <parent link="Right_seg12"/>
+    <child link="Right_seg13"/>
+    <origin xyz="0 0 ${thuind_height}" rpy="0 0 0"/>
+    <axis xyz="0 1 0"/>
+    <dynamics damping="0.7"/>
+    <limit effort="1000.0" lower="0" upper="1.57" velocity="10"/>
+  </joint>
+  <link name="Right_seg13">
+    <collision>
+      <origin xyz="${-x_width/2} 0 ${thuind_height/2}" rpy="0 0 0"/>
+      <geometry>
+         <box size="${x_width} ${imr_width} ${thuind_height}"/>
+      </geometry>
+    </collision>
+    <visual>
+      <origin xyz="${-x_width/2} 0 ${thuind_height/2}" rpy="0 0 0"/>
+      <geometry>
+         <box size="${x_width} ${imr_width} ${thuind_height}"/>
+      </geometry>
+      <material name="black"/>
+    </visual>
+    <inertial>
+      <origin xyz="${-x_width/2} 0 ${thuind_height/2}" rpy="0 0 0"/>
+      <mass value="${mass_palm}"/>
+      <inertia
+    ixx="${mass_palm / 12.0 * (width*width + width*width)}" ixy="0.0" ixz="0.0"
+    iyy="${mass_palm / 12.0 * (length2*length2 + width*width)}" iyz="0.0"
+    izz="${mass_palm / 12.0 * (width*width + length2*length2)}"/>
+    </inertial>
+  </link>
+<!--====================== MIDDLE FINGER ===============================-->
+  <link name="Right_seg21">
+    <collision>
+      <origin xyz="0 0 ${middle_height/2}" rpy="0 0 0"/>
+      <geometry>
+         <box size="${x_width} ${imr_width} 0.2"/>
+      </geometry>
+    </collision>
+    <visual>
+      <origin xyz="0 0 ${middle_height/2}" rpy="0 0 0"/>
+      <geometry>
+         <box size="${x_width} ${imr_width} ${middle_height}"/>
+      </geometry>
+      <material name="orange"/>
+    </visual>
+    <inertial>
+      <origin xyz="0 0 ${middle_height/2}" rpy="0 0 0"/>
       <mass value="${mass_palm}"/>
       <inertia
@@ -648,28 +818,28 @@
     </inertial>
   </link>
-  <joint name="Right_jointt1" type="revolute">
-    <parent link="Right_segt1"/>
-    <child link="Right_segt2"/>
-    <origin xyz="${x_width/2} 0 0.015" rpy="0 0 0"/>
+  <joint name="Right_joint21" type="revolute">
+    <parent link="Right_seg21"/>
+    <child link="Right_seg22"/>
+    <origin xyz="${x_width/2} 0.0 ${middle_height}" rpy="0 0 0"/>
     <axis xyz="0 1 0"/>
     <dynamics damping="0.7"/>
     <limit effort="1000.0" lower="0" upper="1.57" velocity="10"/>
   </joint>
-  <link name="Right_segt2">
-    <collision>
-      <origin xyz="${-x_width/2} 0 ${0.0268/2}" rpy="0 0 0"/>
-      <geometry>
-         <box size="${x_width} 0.021 0.0268"/>
-      </geometry>
-    </collision>
-    <visual>
-      <origin xyz="${-x_width/2} 0 ${0.0268/2}" rpy="0 0 0"/>
-      <geometry>
-         <box size="${x_width} 0.021 0.0268"/>
+  <link name="Right_seg22">
+    <collision>
+      <origin xyz="${-x_width/2} 0 ${middle_height/2}" rpy="0 0 0"/>
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
Commit message: Final Walking model with eye and Laser scanners is ready

File: src/baby/baby_description/urdf/baby.xacro (robot description, xacro)
@@ -4,9 +4,9 @@
   <xacro:property name="PI" value="3.1415926535897931"/>
   <xacro:property name="mass_chest" value="30" />
-  <xacro:property name="mass_palm" value="0.2" /> <!-- arbitrary value for mass -->
+  <xacro:property name="mass_palm" value="0.8" /> <!-- arbitrary value for mass -->
   <xacro:property name="mass_hand" value="05" /> <!-- arbitrary value for mass -->
   <xacro:property name="mass_neck" value="02" />
   <xacro:property name="mass_leg" value="10" />
-  <xacro:property name="mass_foot" value="5" />
+  <xacro:property name="mass_foot" value="30" />
   <xacro:property name="mass_dummy" value="2.0" />
   <!-- Total weight=0.2*8+5*2+10*4+2*1+6*1+5*4+0.2*32+25=1.6+10+40+2+6+20+6.4+25 -->
@@ -20,4 +20,5 @@
   <xacro:property name="chest_width" value="0.05" /><!-- x-->
   <xacro:property name="chest_length" value="0.3" /><!--y-->
+  <xacro:property name="eye_size" value="0.003" />
   <xacro:property name="palm_height" value="0.11" />
   <xacro:property name="palm_length" value="0.1" /> <!--y-->
@@ -39,6 +40,6 @@
   <xacro:property name="leg_radius" value="0.02" />
   <xacro:property name="foot_height" value="0.02" />
-  <xacro:property name="foot_length" value="0.4" />
-  <xacro:property name="foot_width" value="0.4" />
+  <xacro:property name="foot_length" value="0.3" />
+  <xacro:property name="foot_width" value="0.3" />
   <xacro:property name="dummy_size" value="0.10" />
   <xacro:property name="dummy_size_leg" value="0.20" />
@@ -221,5 +222,5 @@
     <axis xyz="0 1 0"/>
     <dynamics damping="0.7"/>
-    <limit effort="1000.0" lower="0" upper="3.14" velocity="10"/>
+    <limit effort="1000.0" lower="-3.14" upper="3.14" velocity="10"/>
   </joint>
   <link name="Left_leg_lower">
@@ -304,5 +305,5 @@
     <axis xyz="0 1 0"/>
     <dynamics damping="0.7"/>
-    <limit effort="1000.0" lower="0" upper="3.14" velocity="10"/>
+    <limit effort="1000.0" lower="-3.14" upper="3.14" velocity="10"/>
   </joint>
   <link name="Right_leg_lower">
@@ -439,4 +440,86 @@
     </inertial>
   </link>
+<!--========================= Eyes =====================================-->
+  <joint name="Left_eye_joint" type="fixed">
+    <axis xyz="0 1 0" />
+    <origin xyz="${head_radius/1.414} ${head_radius/1.414} ${head_height/2}" rpy="0 0 0"/>
+    <parent link="Head"/>
+    <child link="Left_eye"/>
+  </joint>
+  <joint name="Right_eye_joint" type="fixed">
+    <axis xyz="0 1 0" />
+    <origin xyz="${head_radius/1.414} ${-head_radius/1.414} ${head_height/2}" rpy="0 0 0"/>
+    <parent link="Head"/>
+    <child link="Right_eye"/>
+  </joint>
+  <link name="Left_eye">
+    <collision>
+      <origin xyz="0 0 0" rpy="0 0 0"/>
+      <geometry>
+        <box size="${eye_size} ${eye_size} ${eye_size}"/>
+      </geometry>
+    </collision>
+    <visual>
+      <origin xyz="0 0 0" rpy="0 0 0"/>
+      <geometry>
+        <box size="${eye_size} ${eye_size} ${eye_size}"/>
+      </geometry>
+      <material name="red"/>
+    </visual>
+    <inertial>
+      <mass value="1e-5" />
+      <origin xyz="0 0 0" rpy="0 0 0"/>
+      <inertia
+        ixx="1e-6" ixy="0" ixz="0" iyy="1e-6" iyz="0" izz="1e-6" />
+      </inertial>
+  </link>
+  <link name="Right_eye">
+    <collision>
+      <origin xyz="0 0 0" rpy="0 0 0"/>
+      <geometry>
+        <box size="${eye_size} ${eye_size} ${eye_size}"/>
+      </geometry>
+    </collision>
+    <visual>
+      <origin xyz="0 0 0" rpy="0 0 0"/>
+      <geometry>
+        <box size="${eye_size} ${eye_size} ${eye_size}"/>
+      </geometry>
+      <material name="red"/>
+    </visual>
+    <inertial>
+      <mass value="1e-5" />
+      <origin xyz="0 0 0" rpy="0 0 0"/>
+      <inertia
+        ixx="1e-6" ixy="0" ixz="0" iyy="1e-6" iyz="0" izz="1e-6" />
+      </inertial>
+  </link>
+<!--=======================Scanner=======================================-->
+  <joint name="Hokuyo_joint" type="fixed">
+    <axis xyz="0 1 0" />
+    <origin xyz="0 0 ${head_height}" rpy="0 0 0"/>
+    <parent link="Head"/>
+    <child link="Hokuyo_link"/>
+  </joint>
+  <!-- Hokuyo Laser -->
+  <link name="Hokuyo_link">
+    <collision>
+      <origin xyz="0 0 0" rpy="0 0 0"/>
+      <geometry>
+        <box size="${eye_size} ${eye_size} ${eye_size}"/>
+      </geometry>
+    </collision>
+    <visual>
+      <origin xyz="0 0 0" rpy="0 0 0"/>
+      <geometry>
+        <mesh filename="package://baby_description/meshes/hokuyo.dae"/>
+      </geometry>
+    </visual>
+    <inertial>
+      <mass value="1e-5" />
+      <origin xyz="0 0 0" rpy="0 0 0"/>
+      <inertia ixx="1e-6" ixy="0" ixz="0" iyy="1e-6" iyz="0" izz="1e-6" />
+    </inertial>
+  </link>
 <!--======================= 3 axis Right hand ============================-->
   <link name="Right_z_handD">
